File: pcb/KiCad Schematic.sch (KiCad schematic (older format))
At the start: 0 parts

Commit message: add coil winder hardware, code that compiles (for now)
Parts:
- added C1, C12, C13, C4, C5, C6, C8, C9: 100nF, Capacitor_SMD:C_0603_1608Metric, symbol Device:C
- added C10, C11, C3, C7: 1uF, Capacitor_SMD:C_0603_1608Metric, symbol Device:C
- added C14, C17, C2, C31, C34, C35, C36: 10uF, Capacitor_SMD:C_0805_2012Metric, symbol Device:C
- added C15, C16, C30: 47uF, Capacitor_SMD:CP_Elec_6.3x7.7, symbol Device:C
- added C32, C33: 22pF, Capacitor_SMD:C_0603_1608Metric, symbol Device:C
- added D1, D2: LED, LED_SMD:LED_0603_1608Metric, symbol Device:LED
- added D3, D4, D5, D6, D7: CGRTS4004-HF, Diode_SMD:D_SOD-123F, symbol Device:D
- added IC1: AP63205WU-7, SOT95P280X100-6N, symbol SamacSys_Parts:AP63205WU-7
- added IC2: ATSAMD51J19A-MU, Package_DFN_QFN:QFN-64-1EP_9x9mm_P0.5mm_EP6x6mm_ThermalVias, symbol SamacSys_Parts:ATSAMD51J19A-MU
- added J1, J4: PAD, TestPoint:TestPoint_Pad_D2.0mm, symbol Connector_Generic:Conn_01x01
- added J17, J18, J19, J20: Hole, MountingHole:MountingHole_2.7mm_M2.5_DIN965_Pad, symbol Connector_Generic:Conn_01x01
- added J2: Conn_01x02, Connector_BarrelJack:BarrelJack_Wuerth_6941xx301002, symbol Connector_Generic:Conn_01x02
- added J22: Conn_01x06, Connector_PinSocket_2.54mm:PinSocket_1x06_P2.54mm_Vertical, symbol Connector_Generic:Conn_01x06
- added J3: 47346-0001, 47346-0001, symbol SamacSys_Parts:47346-0001
- added J5, J7, J8, J9: Conn_01x02, Connector_PinHeader_2.54mm:PinHeader_1x02_P2.54mm_Vertical, symbol Connector_Generic:Conn_01x02
- added J6: 20021121-00010C4LF, 2002112100010C4LF, symbol SamacSys_Parts:20021121-00010C4LF
- added L1, L2, L3: 10uH, Inductor_SMD:L_0805_2012Metric, symbol Device:L
- added Q1, Q2, Q3, Q4: NVTFS4C08NTAG, NVTFS6H854NTAG, symbol SamacSys_Parts:NVTFS5C680NLTAG
- added R1, R15, R16, R18, R2: 10k, Resistor_SMD:R_0603_1608Metric, symbol Device:R
- added R13, R14, R17, R19, R20, R3, R4: 174, Resistor_SMD:R_0603_1608Metric, symbol Device:R
- added S1: KMR243GLFG, KMR421GULCLFS, symbol SamacSys_Parts:KMR243GLFG
- added U1: TLV493D, Package_TO_SOT_SMD:SOT-23-6, symbol Sensor_Magnetic:TLV493D
- added U3: AP2112K-3.3, Package_TO_SOT_SMD:SOT-23-5, symbol Regulator_Linear:AP2112K-3.3
- added Y1: LFXTAL009678REEL, LFXTAL009678REEL, symbol SamacSys_Parts:LFXTAL009678REEL
Connections:
- net labels added: +3.3V, +5V, +VDC, 3v3, AREF, D+, D-, D0_CS, D0_EN, D0_S0_DIR, D0_S0_STEP, D0_S1_DIR, D0_S1_STEP, D1_CS, D1_EN, D1_S0_DIR, D1_S0_STEP, D1_S1_DIR, D1_S1_STEP, GATE0, GATE1, GEN0, GEN1, GEN10, GEN11, GEN12, GEN13, GEN14, GEN2, GEN3, GEN4, GEN5, GEN6, GEN7, GEN8, GEN9, GND, MISO, MOSI, OSC0, OSC1, RESET, RX, SCK, SCL, SDA, SD_CS, SERVO0, SERVO1, SERVO2, SWCLK, SWDIO, TX, VDDCORE, VSENSE, VSW, gnd
- wire segments 0 -> 363
Other:
- note added: "COMS I/O"
- note added: "FET GATES"
- note added: "GPIO"
- note added: "MAG SENSOR\n"
- note added: "MCU"
- note added: "POWER FILTERING"
- note added: "POWER REG"
- note added: "PROG HEADER"
- note added: "STATUS"
